File: PCB/swipe-stack-glove/swipe-stack-glove.kicad_sch (KiCad schematic)
At the start: 48 parts, among them J1 Conn_02x05_Odd_Even, J2 Conn_01x05_Socket, J3 Conn_01x01_Pin, J4 Conn_01x01_Pin, J5 Conn_01x01_Pin, SW1 SW_Push, SW2 SW_Push, SW3 SW_Push, SW4 SW_Push, U1 STM32F091RCTx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

Commit message: Latest glove pcb
Parts:
- removed J1: Conn_02x05_Odd_Even, Connector_IDC:IDC-Header_2x05_P2.54mm_Vertical, symbol Connector_Generic:Conn_02x05_Odd_Even
- added C14: 0.1uF, Capacitor_SMD:C_0805_2012Metric_Pad1.18x1.45mm_HandSolder, symbol Device:C
- added J6: Conn_01x04, Connector_PinHeader_2.54mm:PinHeader_1x04_P2.54mm_Vertical, symbol Connector_Generic:Conn_01x04
- SW1, SW2, SW3, SW4: footprint Button_Switch_SMD:SW_SPST_PTS645 -> Button_Switch_SMD:SW_SPST_Omron_B3FS-100xP
Connections:
- net +3.3V: now also C14.1
- net GND: now also C14.2, J6.2 (Pin_2); no longer U2.14 (INT)
- net IMU_RX: now also U2.19 (COM1); no longer U2.20 (COM0)
- net IMU_TX: now also U2.20 (COM0); no longer U2.19 (COM1)
- net NRST: now also J6.1 (Pin_1)
- net SWCLK_IN: now also J6.3 (Pin_3)
- net SWDIO_IN: now also J6.4 (Pin_4)
- no-connect marks 57 -> 53
Other:
- note added: "32KHz crystal"
- note added: "8MHz oscillator"
- note added: "Bluetooth"
- note added: "Boot pin"
- note added: "Debug LEDs"
- note added: "Debug buttons"
- note added: "Decoupling capacitors"
- note added: "IMU"
- note added: "Microcontroller"
- note added: "Mounting holes"
- note added: "Programming header"
- note added: "Reset button"
- note added: "Voltage regulator"
- note removed: "Author: Aditya Sood"
- note removed: "TODO: heartbeat LED supply decaps extra GPIO"
- moved on the sheet: C10, C11, C12, C13, C2, C3, C4, C5, C9, D1, D2, H1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
