File: PCB/swipe-stack-glove/swipe-stack-glove.kicad_pcb (KiCad board)
At the start: 2 copper layers, 63.1 x 63.2 mm, 46 parts, among them J1 Conn_02x05_Odd_Even, J2 Conn_01x05_Socket, J3 Conn_01x01_Pin, J4 Conn_01x01_Pin, J5 Conn_01x01_Pin, SW1 SW_Push, SW2 SW_Push, SW3 SW_Push, SW4 SW_Push, U1 STM32F091RCTx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

Commit message: Latest glove pcb
Parts:
- removed J1: Conn_02x05_Odd_Even, Connector_IDC:IDC-Header_2x05_P2.54mm_Vertical
- removed U5: Adafruit Charger, GlovePCB:AdaFruit Charger
- removed U6: BatteryCell, GlovePCB:battery_cell
- added C14: 0.1uF, Capacitor_SMD:C_0805_2012Metric_Pad1.18x1.45mm_HandSolder, F.Cu at (142.7, 107.2)
- added H2: B_TopRight, MountingHole:MountingHole_2.5mm, F.Cu at (167.8, 75.9)
- added J6: Conn_01x04, Connector_PinHeader_2.54mm:PinHeader_1x04_P2.54mm_Vertical, B.Cu at (135.4, 86.0)
- D1, R2, R3, R4: moved to B.Cu
- SW1, SW3, SW4: footprint Button_Switch_SMD:SW_SPST_PTS645 -> Button_Switch_SMD:SW_SPST_Omron_B3FS-100xP
- SW2: footprint Button_Switch_SMD:SW_SPST_PTS645 -> Button_Switch_SMD:SW_SPST_Omron_B3FS-100xP; moved to B.Cu
- moved C2 143.9 mm to (166.2, 92.7), turned to 180 degrees
- moved C11 106.1 mm to (158.2, 110.5), turned to 180 degrees
- moved C12 98.9 mm to (160.0, 96.3)
- moved C9 98.0 mm to (147.1, 94.0), turned to 90 degrees
- moved C10 93.1 mm to (149.2, 111.3), turned to 180 degrees
- moved J2 81.5 mm to (151.8, 123.9), turned to 90 degrees
- moved D2 80.2 mm to (155.7, 118.5), turned to 0 degrees
- moved R7 79.7 mm to (160.3, 118.5), turned to 180 degrees
- moved C13 78.7 mm to (144.0, 98.1), turned to 90 degrees
- moved H4 63.7 mm to (167.9, 122.7)
- moved H3 60.3 mm to (136.4, 122.7)
- moved SW2 54.9 mm to (165.1, 103.6), turned to -90 degrees
- moved R4 51.6 mm to (169.8, 95.0)
- moved SW3 48.6 mm to (145.7, 118.9), turned to 180 degrees
- moved D1 47.0 mm to (166.3, 95.9), turned to 0 degrees
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Connections:
- U2 pad 14: GND -> unconnected-(U2-INT-Pad14)
- U2 pad 19: /IMU_TX -> /IMU_RX
- U2 pad 20: /IMU_RX -> /IMU_TX
Routing:
- net +3.3V: track 45.5 -> 134.7 mm, vias 0 -> 15
- net /NRST: track 70.5 -> 35.6 mm, vias 3 -> 4
- net Net-(U4-PIO1): track 5.38 -> 25.3 mm, vias 0 -> 1
- net Net-(U4-PIO0): track 16.6 -> 36.5 mm, vias 0 -> 1
- net Net-(R12-Pad2): track 2.83 -> 20.4 mm
- net /EXTRA3: track 10.6 -> 21.7 mm, vias 0 -> 2
- net /IMU_RX: track 21.9 -> 12.2 mm
- net /SWCLK_IN: track 33.8 -> 24.1 mm
- net Net-(U4-BX_RX): track 18.6 -> 9.75 mm, vias 0 -> 1
- net /PB2: track 10.4 -> 2.89 mm, vias 2 -> 0
- net /IMU_TX: track 19.1 -> 13.1 mm, vias 2 -> 0
- net /PC8: track 4.03 -> 9.84 mm
- net /BOOT0: track 4.70 -> 10.4 mm
- net /B_TX: track 11.7 -> 16.8 mm, vias 0 -> 1
- net Net-(U4-BX_TX): track 20.0 -> 15.1 mm, vias 0 -> 1
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- added copper zone on B.Cu, net +3.3V
- added copper zone on F.Cu, net GND
- removed copper zone on F.Cu, net +3.3V
- removed copper zone on B.Cu, net GND
Other:
- board size 63.1 x 63.2 mm -> 38.1 x 53.3 mm
- board text added: "Team 13: Glove PCB Aditya S. Alex C. Justin C. Vishnu L."

Commit message: gerber done
Parts:
- moved D1 15.4 mm to (168.8, 111.1), turned to 90 degrees
- moved R4 10.5 mm to (168.8, 105.5)
- moved SW2 6.30 mm to (160.4, 107.8), turned to 0 degrees
- moved C4 4.87 mm to (167.9, 96.0), turned to 90 degrees
- moved C5 4.45 mm to (167.9, 100.5)
- moved XTAL1 2.63 mm to (164.8, 98.2), turned to -90 degrees
- moved J5 1.30 mm to (167.7, 117.8)
- moved C2 0.95 mm to (166.3, 91.7)
- moved C3 0.79 mm to (166.4, 86.2)
- moved J4 0.24 mm to (135.4, 81.0)
Routing:
- net Net-(U4-PIO0): track 36.5 -> 60.0 mm
- net Net-(U4-PIO1): track 25.3 -> 43.3 mm
- net GND: track 58.6 -> 68.1 mm, vias 2 -> 5
- net /XOUT32: track 10.4 -> 14.9 mm
- net Net-(U4-BX_RX): track 9.75 -> 12.9 mm
- net /SWDIO_IN: track 30.0 -> 32.9 mm
- net /EXTRA3: track 21.7 -> 23.1 mm
- net Net-(D1-A): track 2.48 -> 3.65 mm
- net +3.3V: track 134.7 -> 134.5 mm, vias 15 -> 14
